Commit message: test environment

File: src/ur_robotiq/ur_robotiq_description/urdf/ur_robotiq.urdf.xacro (robot description, xacro)
@@ -8,5 +8,5 @@
     <parent link="world" />
     <child link = "base_link" />
-    <origin xyz="0.0 0.0 0.0" rpy="0.0 0.0 0.0" />
+    <origin xyz="0.0 0.0 0.5" rpy="0.0 0.0 ${pi}" />
   </joint>
   <xacro:robotiq_85_gripper prefix="" parent="wrist_3_link" >

Commit message: moveit rviz

File: src/ur_robotiq/ur_robotiq_description/urdf/ur_robotiq.urdf.xacro (robot description, xacro)
@@ -5,5 +5,5 @@
   <xacro:ur5_robot prefix="" joint_limited="false"/>
   <link name="world" />
-  <joint name="world_joint" type="fixed">
+  <joint name="fixed_base" type="fixed">
     <parent link="world" />
     <child link = "base_link" />

Commit message: fix bug

File: src/ur_robotiq/ur_robotiq_description/urdf/ur_robotiq.urdf.xacro (robot description, xacro)
@@ -1,12 +1,13 @@
 <?xml version="1.0"?>
 <robot xmlns:xacro="http://www.ros.org/wiki/xacro" name="ur_robotiq">
+  <xacro:include filename="$(find ur_description)/urdf/common.gazebo.xacro" />
   <xacro:include filename="$(find ur_description)/urdf/ur5.urdf.xacro" />
   <xacro:include filename="$(find robotiq_85_description)/urdf/robotiq_85_gripper.urdf.xacro" />
   <xacro:ur5_robot prefix="" joint_limited="false"/>
   <link name="world" />
-  <joint name="fixed_base" type="fixed">
+  <joint name="world_joint" type="fixed">
     <parent link="world" />
     <child link = "base_link" />
-    <origin xyz="0.0 0.0 0.5" rpy="0.0 0.0 ${pi}" />
+    <origin xyz="0.0 0.0 0.7" rpy="0.0 0.0 0.0" />
   </joint>
   <xacro:robotiq_85_gripper prefix="" parent="wrist_3_link" >

Commit message: add kinectv2

File: src/ur_robotiq/ur_robotiq_description/urdf/ur_robotiq.urdf.xacro (robot description, xacro)
@@ -4,4 +4,6 @@
   <xacro:include filename="$(find ur_description)/urdf/ur5.urdf.xacro" />
   <xacro:include filename="$(find robotiq_85_description)/urdf/robotiq_85_gripper.urdf.xacro" />
+  <xacro:include filename="$(find pr2_description)/urdf/common.xacro" />
+  <xacro:include filename="$(find pr2_description)/urdf/sensors/kinect2.urdf.xacro" />
   <xacro:ur5_robot prefix="" joint_limited="false"/>
   <link name="world" />
@@ -14,3 +16,6 @@
     <origin xyz="0 0.1 0" rpy="0 0 ${pi/2}"/>
   </xacro:robotiq_85_gripper>
+  <xacro:kinect2_v0 name="" parent="world" >
+    <origin xyz="0.4 0.0 1.2" rpy="0.0 ${pi/2} 0.0" />
+  </xacro:kinect2_v0>
 </robot>
